File: Daughterboard.kicad_pcb (KiCad board)
At the start: 4 copper layers, 285.8 x 94.6 mm, 90 parts, among them CN451 Video_Slot, CN452 Video_Slot, CN600 Zorro-III, CN601 Zorro-III, CN602 Zorro-III, CN603 Zorro-III, CN751 ISA_8_Bit, CN752 ISA_8_Bit, CN754 ISA_16_Bit_Extended, CN755 ISA_16_Bit_Extended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

Commit message: Amended Layout to resolve potential short and move upper notch
Routing:
- net +12V: track 513.0 -> 512.1 mm
Other:
- outline, holes or cut-outs redrawn
